File: mSolarWeather.kicad_sch (KiCad schematic)
At the start: 66 parts, among them J1 Solar connector, J2 JST2PH Batt LiFePo4 3.2v, J3 USB C, J4 I2C ext, J5 Micro_SD_Card_Det_Hirose_DM3AT, J6 LUX_I2C module, J7 BME280_I2C module, J8 WIND, J9 RAIN, SW1 SW_Push_Dual, SW2 SW_Push_Dual, U1 TPS63021, U2 BQ25185, U3 ESP32-S3-WROOM-1-N16R2, U4 Ai-Thinker-Ra-01, U5 DS3231MZ

Commit message: Update diagram
Parts:
- removed D2: LED PSupply, LED_SMD:LED_PLCC-2_3.4x3.0mm_KA, symbol Device:LED
- removed J5: Micro_SD_Card_Det_Hirose_DM3AT, Connector_Card:microSD_HC_Hirose_DM3AT-SF-PEJM5, symbol Connector:Micro_SD_Card_Det_Hirose_DM3AT
- removed R2: 4.7k, Resistor_SMD:R_0805_2012Metric_Pad1.20x1.40mm_HandSolder, symbol Device:R
- added C16: 22uF, symbol Device:C
- added D10: LED PSupply, LED_SMD:LED_PLCC-2_3.4x3.0mm_KA, symbol Device:LED
- added F2, F3: Polyfuse xA, symbol Device:Polyfuse_Small
- added J10: Micro_SD_Card, symbol Connector:Micro_SD_Card
- added Q1, Q2: PMOS, symbol Simulation_SPICE:PMOS
- added R18, R20: 10k, Resistor_SMD:R_0805_2012Metric_Pad1.20x1.40mm_HandSolder, symbol Device:R
- added R21: 4.7k, Resistor_SMD:R_0805_2012Metric_Pad1.20x1.40mm_HandSolder, symbol Device:R
- C2: value 22uF -> 100nF; footprint (none) -> Capacitor_SMD:C_0805_2012Metric_Pad1.18x1.45mm_HandSolder; Fournisseur (none) -> RS: 648-0941
- R8: value 422k -> 22k
- R9: value 160 -> 100k
Connections:
- net +3.3V: now also Q1.3 (S), Q2.3 (S), R18.2, R20.2
- net GND: now also C2.1, C16.2, D10.1 (K), J10.6 (VSS), J10.9 (SHIELD); no longer C2.2
- net I2C_PWR: now also R1.1, F2.2; no longer C2.1
- net SD_PWR: now also F3.2, J10.4 (VDD), R21.1; no longer C1.1, R1.1
- net cmd_I2C_PWR: now also Q1.2 (G), R18.1
- net cmd_SD_PWR: now also Q2.2 (G), R20.1
- net at R8.2, R9.1, U3.39 (IO1): now also C2.2
- new net: C1.1, F2.1, Q1.1 (D)
- new net: C16.1, F3.1, Q2.1 (D)
- new net: D10.2 (A), R21.2
Other:
- note added: "1.8 V to 5.5 V"
- moved on the sheet: C1, C10, D1, F1, J2, R1, R8, R9, U3
