File: mSolarWeather.kicad_sch (KiCad schematic)
At the start: 47 parts, among them J1 USB_C_USB2.0, J2 Micro_SD_Card, J3 Debug 1, J4 Debug 2, J5 LUX_I2C module, J6 BME280_I2C module, J7 WIND, J8 RAIN, J9 I2C ext, SW1 SW_Push_Dual, SW2 SW_Push_Dual, SW3 SW_Push_Dual, U1 DS3231MZ, U2 Ai-Thinker-Ra-01, U3 USBLC6-2SC6, U4 ESP32-S3-WROOM-1-N16R2

Commit message: update and starting PCB
Parts:
- removed D5: ESD3.3, Diode_SMD:D_SOD-923, symbol Diode:ESD9B3.3ST5G
- removed H1, H2, H3, H4: MountingHole, MountingHole:MountingHole_3.2mm_M3, symbol Mechanical:MountingHole
- removed SW1, SW2, SW3: SW_Push_Dual, Button_Switch_SMD:SW_Push_1P1T_NO_CK_KSC9xxG, symbol Switch:SW_Push_Dual
- added D4: ESD3.3, Diode_SMD:D_SOD-923, symbol Diode:ESD9B3.3ST5G
- added H1, H2, H3, H4: MountingHole_Pad, MountingHole:MountingHole_3.2mm_M3_Pad_Via, symbol Mechanical:MountingHole_Pad
- added SW1: SW_boot, Button_Switch_SMD:SW_Push_1P1T_NO_CK_KSC9xxG, symbol Switch:SW_Push
- added SW2: SW_rst, Button_Switch_SMD:SW_Push_1P1T_NO_CK_KSC9xxG, symbol Switch:SW_Push
- added SW3: SW_user, Button_Switch_SMD:SW_Push_1P1T_NO_CK_KSC9xxG, symbol Switch:SW_Push
- renumbered D4 to D5
Connections:
- net Boot: now also SW1.2
- net Btn_User: now also D4.2 (A2), SW3.2
- net GND: now also D4.1 (A1), H1.1, H2.1, H3.1, H4.1, SW1.1, SW2.1, SW3.1
- net Reset: now also SW2.2
Other:
- moved on the sheet: C5, D2, D3, R6
