File: mSolarWeather.kicad_pcb (KiCad board)
At the start: 2 copper layers, 55 parts, among them J1 Solar connector, J2 JST2PH Batt LiFePo4 3.2v, J3 USB C, J4 I2C ext, J5 Micro_SD_Card_Det_Hirose_DM3AT, J6 LUX_I2C module, J7 BME280_I2C module, J8 WIND, J9 RAIN, U1 TPS63021, U2 BQ25185, U3 ESP32-S3-WROOM-1-N16R2, U4 Ai-Thinker-Ra-01, U5 DS3231MZ

Commit message: update and starting PCB
Parts:
- added C1: 10uF, Capacitor_SMD:C_1206_3216Metric_Pad1.33x1.80mm_HandSolder, F.Cu at (63.2, 85.8)
- added C12: 10uF, Capacitor_SMD:C_1206_3216Metric_Pad1.33x1.80mm_HandSolder, F.Cu at (101.7, 48.7)
- added C16: 22uF, Capacitor_SMD:C_1210_3225Metric_Pad1.33x2.70mm_HandSolder, F.Cu at (77.4, 24.6)
- added C17: 22uF, Capacitor_SMD:C_1210_3225Metric_Pad1.33x2.70mm_HandSolder, F.Cu at (77.4, 28.9)
- added C18: 22uF, Capacitor_SMD:C_Elec_5x5.4, F.Cu at (99.2, 21.7)
- added C19: 22uF, Capacitor_SMD:C_1210_3225Metric_Pad1.33x2.70mm_HandSolder, F.Cu at (77.4, 33.1)
- added C2: 100nF, Capacitor_SMD:C_0805_2012Metric_Pad1.18x1.45mm_HandSolder, F.Cu at (57.5, 19.8)
- added C20: 22uF, Capacitor_SMD:C_1210_3225Metric_Pad1.33x2.70mm_HandSolder, F.Cu at (77.4, 37.4)
- added C21: 22uF, Capacitor_SMD:C_1210_3225Metric_Pad1.33x2.70mm_HandSolder, F.Cu at (77.4, 41.6)
- added C3: 100nF, Capacitor_SMD:C_0805_2012Metric_Pad1.18x1.45mm_HandSolder, F.Cu at (57.5, 22.8)
- added C4: 100nF, Capacitor_SMD:C_0805_2012Metric_Pad1.18x1.45mm_HandSolder, F.Cu at (57.5, 25.8)
- added C5: 1uF, Capacitor_SMD:C_0805_2012Metric_Pad1.18x1.45mm_HandSolder, F.Cu at (57.5, 28.8)
- added C7: 100nF, Capacitor_SMD:C_0805_2012Metric_Pad1.18x1.45mm_HandSolder, F.Cu at (57.5, 31.8)
- added C8: 1uF, Capacitor_SMD:C_0805_2012Metric_Pad1.18x1.45mm_HandSolder, F.Cu at (57.5, 34.8)
- added C9: 1uF, Capacitor_SMD:C_0805_2012Metric_Pad1.18x1.45mm_HandSolder, F.Cu at (57.5, 37.8)
- added D10: LED PSupply, LED_SMD:LED_PLCC-2_3.4x3.0mm_KA, F.Cu at (71.4, 29.6)
- added D11: LED PSupply, LED_SMD:LED_PLCC-2_3.4x3.0mm_KA, F.Cu at (71.4, 34.2)
- added D12: LED PSupply, LED_SMD:LED_PLCC-2_3.4x3.0mm_KA, F.Cu at (71.4, 38.7)
- added D13: LED PSupply, LED_SMD:LED_PLCC-2_3.4x3.0mm_KA, F.Cu at (71.4, 43.3)
- added F1: Polyfuse 2.6A, Fuse:Fuse_1206_3216Metric, F.Cu at (92.2, 19.9)
- added F2: Polyfuse 1.5A, Fuse:Fuse_1206_3216Metric, F.Cu at (92.2, 23.2)
- added F3: Polyfuse 1.5A, Fuse:Fuse_1206_3216Metric, F.Cu at (92.2, 26.5)
- added F4: Polyfuse 1.5A, Fuse:Fuse_1206_3216Metric, F.Cu at (92.2, 29.8)
- added J10: JST2PH Batt LiFePo4 3.2v, Connector_JST:JST_PH_S2B-PH-K_1x02_P2.00mm_Horizontal, F.Cu at (99.6, 34.0)
- added J11: Solar connector, TerminalBlock_Phoenix:TerminalBlock_Phoenix_MKDS-1,5-2-5.08_1x02_P5.08mm_Horizontal, F.Cu at (92.2, 96.7)
- added Q1: IRLML6401, Package_TO_SOT_SMD:SOT-23, F.Cu at (86.9, 20.5)
- added Q2: IRLML6401, Package_TO_SOT_SMD:SOT-23, F.Cu at (86.9, 24.9)
- added Q3: IRLML6401, Package_TO_SOT_SMD:SOT-23, F.Cu at (86.9, 29.4)
- added R20: 10k, Resistor_SMD:R_0805_2012Metric_Pad1.20x1.40mm_HandSolder, F.Cu at (96.3, 45.2)
- added R21: 4.7k, Resistor_SMD:R_0805_2012Metric_Pad1.20x1.40mm_HandSolder, F.Cu at (96.3, 48.1)
- added R22: 4.7k, Resistor_SMD:R_0805_2012Metric_Pad1.20x1.40mm_HandSolder, F.Cu at (96.3, 51.1)
- added R23: 4.7k, Resistor_SMD:R_0805_2012Metric_Pad1.20x1.40mm_HandSolder, F.Cu at (96.3, 54.0)
- added SW1: SW_boot, Button_Switch_SMD:SW_Push_1P1T_NO_CK_KSC9xxG, F.Cu at (13.0, 64.4)
- added SW2: SW_rst, Button_Switch_SMD:SW_Push_1P1T_NO_CK_KSC9xxG, F.Cu at (13.0, 72.1)
- added SW3: SW_user, Button_Switch_SMD:SW_Push_1P1T_NO_CK_KSC9xxG, F.Cu at (13.0, 79.9)
- added TP1: VBatt, TestPoint:TestPoint_Pad_D2.0mm, F.Cu at (82.4, 20.3)
- added TP2: 3.3V, TestPoint:TestPoint_Pad_D2.0mm, F.Cu at (82.4, 24.3)
- added TP3: SD_PWR, TestPoint:TestPoint_Pad_D2.0mm, F.Cu at (82.4, 28.4)
- added TP4: I2C_PWR, TestPoint:TestPoint_Pad_D2.0mm, F.Cu at (82.4, 32.4)
- added TP5: Lora_PWR, TestPoint:TestPoint_Pad_D2.0mm, F.Cu at (82.4, 36.5)
- added U6: BQ25185, Package_SON:WSON-10-1EP_2.5x2.5mm_P0.5mm_EP1.2x2mm_ThermalVias, F.Cu at (71.1, 47.6)
- BT1: value 2032 -> CR1220; footprint Battery:BatteryHolder_MYOUNG_BS-07-A1BJ001_CR2032 -> Battery:BatteryHolder_Keystone_500
- C10: value 100nF -> 1uF
- C11: value 1uF -> 10uF; footprint Capacitor_SMD:C_0805_2012Metric_Pad1.18x1.45mm_HandSolder -> Capacitor_SMD:C_1206_3216Metric_Pad1.33x1.80mm_HandSolder
- C13: value 100nF -> 10uF; footprint Capacitor_SMD:C_0805_2012Metric_Pad1.18x1.45mm_HandSolder -> Capacitor_SMD:C_1206_3216Metric_Pad1.33x1.80mm_HandSolder
- C15, C6: value 100nF -> 22uF; footprint Capacitor_SMD:C_0805_2012Metric_Pad1.18x1.45mm_HandSolder -> Capacitor_SMD:C_1210_3225Metric_Pad1.33x2.70mm_HandSolder
- D2: value LED PSupply -> ESD3.3; footprint LED_SMD:LED_PLCC-2_3.4x3.0mm_KA -> Diode_SMD:D_SOD-923
- D3, D4: value NSR0320 -> ESD3.3; footprint Diode_SMD:D_SOD-323_HandSoldering -> Diode_SMD:D_SOD-923
- D5: value LED PSupply -> LED RGB NeoPixel; footprint LED_SMD:LED_PLCC-2_3.4x3.0mm_KA -> LED_SMD:LED_Inolux_IN-PI554FCH_PLCC4_5.0x5.0mm_P3.2mm
- D6: value FAULT Red -> NSR0320; footprint LED_SMD:LED_PLCC-2_3.4x3.0mm_KA -> Diode_SMD:D_SOD-323_HandSoldering
- D7: value CHG Orange -> NSR0320; footprint LED_SMD:LED_PLCC-2_3.4x3.0mm_KA -> Diode_SMD:D_SOD-323_HandSoldering
- D8: value LED RGB NeoPixel -> FAULT Red; footprint LED_SMD:LED_Inolux_IN-PI554FCH_PLCC4_5.0x5.0mm_P3.2mm -> LED_SMD:LED_PLCC-2_3.4x3.0mm_KA
- D9: value LED PSupply -> CHG Orange
- FB1: footprint Inductor_SMD:L_0805_2012Metric_Pad1.15x1.40mm_HandSolder -> Inductor_SMD:L_0805_2012Metric_Pad1.05x1.20mm_HandSolder
- H1, H2, H3, H4: value MountingHole -> MountingHole_Pad; footprint MountingHole:MountingHole_3.2mm_M3 -> MountingHole:MountingHole_3.2mm_M3_Pad_Via
- J1: value Solar connector -> USB_C_USB2.0; footprint TerminalBlock_Phoenix:TerminalBlock_Phoenix_MKDS-1,5-2-5.08_1x02_P5.08mm_Horizontal -> Connector_USB:USB_C_Receptacle_Palconn_UTC16-G
- J2: value JST2PH Batt LiFePo4 3.2v -> Micro_SD_Card; footprint Connector_JST:JST_PH_S2B-PH-K_1x02_P2.00mm_Horizontal -> Connector_Card:microSD_HC_Hirose_DM3AT-SF-PEJM5
- J3: value USB C -> Debug 1; footprint Connector_USB:USB_C_Receptacle_GCT_USB4105-xx-A_16P_TopMnt_Horizontal -> Connector_PinHeader_2.54mm:PinHeader_1x06_P2.54mm_Vertical
- J4: value I2C ext -> Debug 2; footprint TerminalBlock_Phoenix:TerminalBlock_Phoenix_MKDS-1,5-4-5.08_1x04_P5.08mm_Horizontal -> Connector_PinHeader_2.54mm:PinHeader_1x06_P2.54mm_Vertical
- J5: value Micro_SD_Card_Det_Hirose_DM3AT -> LUX_I2C module; footprint Connector_Card:microSD_HC_Hirose_DM3AT-SF-PEJM5 -> Connector_JST:JST_SH_SM04B-SRSS-TB_1x04-1MP_P1.00mm_Horizontal
- J6: value LUX_I2C module -> BME280_I2C module
- J7: value BME280_I2C module -> WIND; footprint Connector_JST:JST_SH_SM04B-SRSS-TB_1x04-1MP_P1.00mm_Horizontal -> Connector_RJ:RJ14_Connfly_DS1133-S4_Horizontal
- J8: value WIND -> RAIN
- J9: value RAIN -> I2C ext; footprint Connector_RJ:RJ14_Connfly_DS1133-S4_Horizontal -> TerminalBlock_Phoenix:TerminalBlock_Phoenix_MKDS-1,5-4-5.08_1x04_P5.08mm_Horizontal
- L1: footprint Inductor_SMD_Wurth:L_Wurth_WE-LQSH-2010 -> Inductor_SMD_Wurth:L_Wurth_WE-LQSH-4020
- R1, R2: value 4.7k -> 5.1k
- R11: value 600 -> 4.7k
- R12: value 5.1K -> 10k
- R14: value 10k -> 600
- R15: value 3.3k -> 5.1K
- R16: value 3.3k -> 10k
- R17: value 10k -> 4.7k
- R3: value 5.1k -> 5.1K
- R4: value 5.1K -> 22k
- R5: value 5.1k -> 100k
- R8: value 422k -> 10k
- R9: value 160 -> 10k
- U1: value TPS63021 -> DS3231MZ; footprint mSolarLib:VSON_DSJ-14-3x4mm_P0.5mm_ThermalVias -> Package_SO:SOIC-8_3.9x4.9mm_P1.27mm
- U2: value BQ25185 -> Ai-Thinker-Ra-01; footprint Package_SON:WSON-10-1EP_2.5x2.5mm_P0.5mm_EP1.2x2mm_ThermalVias -> RF_Module:Ai-Thinker-Ra-01-LoRa
- U3: value ESP32-S3-WROOM-1-N16R2 -> USBLC6-2SC6; footprint RF_Module:ESP32-S3-WROOM-1 -> Package_TO_SOT_SMD:SOT-23-6
- U4: value Ai-Thinker-Ra-01 -> ESP32-S3-WROOM-1-N16R2; footprint RF_Module:Ai-Thinker-Ra-01-LoRa -> RF_Module:ESP32-S3-WROOM-1
- U5: value DS3231MZ -> TPS63021; footprint Package_SO:SOIC-8_3.9x4.9mm_P1.27mm -> mSolarLib:VSON_DSJ-14-3x4mm_P0.5mm_ThermalVias
- moved U1 153.8 mm to (24.0, 93.1)
- moved J9 146.6 mm to (23.4, 66.7)
- moved D8 140.8 mm to (71.4, 20.5)
- moved D3 140.6 mm to (37.8, 92.7)
- moved D4 140.5 mm to (37.8, 94.6)
- moved C15 139.3 mm to (77.4, 20.4)
- moved C10 137.0 mm to (57.5, 40.8)
- moved J1 135.3 mm to (12.0, 87.9)
- moved C14 124.7 mm to (70.7, 51.1)
- moved J3 124.6 mm to (44.5, 81.8)
- moved C6 116.8 mm to (63.2, 89.6)
- moved U5 114.9 mm to (96.5, 26.4)
- moved J4 112.6 mm to (49.1, 81.8)
- moved D9 108.9 mm to (71.4, 25.1)
- moved D5 105.6 mm to (32.3, 93.0)
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Connections:
- C10 pad 2: +3.3V -> /rain_sensor
- C11 pad 1: /Reset -> Net-(D6-A)
- C13 pad 1: GND -> VS
- C13 pad 2: +3.3V -> GND
- C14 pad 1: GND -> Net-(U5-EN)
- C14 pad 2: /wind_speed -> GND
- C15 pad 1: GND -> Net-(U5-FB)
- C15 pad 2: /rain_sensor -> GND
- C6 pad 1: Net-(U1-EN) -> GND
- C6 pad 2: GND -> +3.3V
- D2 pad 2: Net-(D2-A) -> /Boot
- D3 pad 1: (no net) -> GND
- D3 pad 2: (no net) -> /Reset
- D4 pad 1: (no net) -> GND
- D4 pad 2: (no net) -> /Btn_User
- D5 pad 2: Net-(D5-A) -> /neoPixel
- D6 pad 2: VS -> Net-(D6-A)
- D7 pad 1: Net-(D7-K) -> Net-(D6-K)
- D7 pad 2: VS -> VBUS
- D8 pad 1: GND -> Net-(D8-K)
- D8 pad 2: /neoPixel -> VS
- D9 pad 1: GND -> Net-(D9-K)
- D9 pad 2: Net-(D9-A) -> VS
- FB1 pad 1: Net-(U1-FB) -> Net-(U5-FB)
- J2 pad 1: Net-(J2-Pin_1) -> unconnected-(J2-DAT2-Pad1)
- J2 pad 2: GND -> /CS_SD
- J4 pad 1: /SCL -> /wind_dir
- J4 pad 2: /SDA -> /wind_speed
- J4 pad 3: /I2C_PWR -> /rain_sensor
- J4 pad 4: GND -> /IRQ_DS
- J5 pad 1: unconnected-(J5-DAT2-Pad1) -> /SCL
- J5 pad 2: unconnected-(J5-DAT3/CD-Pad2) -> /SDA
- J5 pad 3: unconnected-(J5-CMD-Pad3) -> I2C_PWR
- J5 pad 4: /SD_PWR -> GND
- J6 pad 1: unconnected-(J6-Pin_1-Pad1) -> /SCL
- J6 pad 2: unconnected-(J6-Pin_2-Pad2) -> /SDA
- J6 pad 3: unconnected-(J6-Pin_3-Pad3) -> I2C_PWR
- J6 pad 4: unconnected-(J6-Pin_4-Pad4) -> GND
- J7 pad 1: unconnected-(J7-Pin_1-Pad1) -> GND
- J7 pad 2: unconnected-(J7-Pin_2-Pad2) -> GND
- J7 pad 3: unconnected-(J7-Pin_3-Pad3) -> /wind_speed
- J7 pad 4: unconnected-(J7-Pin_4-Pad4) -> /wind_dir
- J8 pad 1: GND -> unconnected-(J8-Pad1)
- J8 pad 3: /wind_speed -> /rain_sensor
- J8 pad 4: /wind_dir -> unconnected-(J8-Pad4)
- J9 pad 1: unconnected-(J9-Pad1) -> /SCL
- J9 pad 2: GND -> /SDA
- J9 pad 3: /rain_sensor -> I2C_PWR
- J9 pad 4: unconnected-(J9-Pad4) -> GND
- R1 pad 1: /SD_PWR -> Net-(J1-CC2)
- R1 pad 2: Net-(D1-A) -> GND
- R10 pad 1: +3.3V -> I2C_PWR
- R10 pad 2: Net-(D9-A) -> /SCL
- R11 pad 1: /ISET -> I2C_PWR
- R11 pad 2: GND -> /SDA
- R12 pad 1: /ILIM/VSET -> Net-(D8-K)
- R12 pad 2: GND -> Net-(U6-STAT1)
- R13 pad 1: /THERM -> Net-(D9-K)
- R13 pad 2: GND -> Net-(U6-STAT2)
- R14 pad 1: +3.3V -> /Power Management/ISET
- R14 pad 2: /Reset -> GND
- R15 pad 1: +3.3V -> /Power Management/ILIM/VSET
- R15 pad 2: /SDA -> GND
- R16 pad 1: +3.3V -> /Power Management/THERM
- R16 pad 2: /SCL -> GND
- R17 pad 2: /wind_dir -> Net-(D10-A)
- R18 pad 1: +3.3V -> /cmd_SD_PWR
- R18 pad 2: /wind_speed -> +3.3V
- R19 pad 1: +3.3V -> /cmd_I2C_PWR
- R19 pad 2: /rain_sensor -> +3.3V
- R2 pad 1: /I2C_PWR -> Net-(J1-CC1)
- R2 pad 2: Net-(D2-A) -> GND
- R3 pad 1: Net-(J3-CC2) -> VBUS
- R3 pad 2: GND -> Net-(D1-A)
- R4 pad 1: VBUS -> +BATT
- R4 pad 2: Net-(D5-A) -> Net-(U4-IO1)
- R5 pad 1: Net-(J3-CC1) -> Net-(U4-IO1)
- R6 pad 1: Net-(D6-K) -> +3.3V
- R6 pad 2: Net-(U2-STAT1) -> /Reset
- R7 pad 1: Net-(D7-K) -> +3.3V
- R7 pad 2: Net-(U2-STAT2) -> /Btn_User
- R8 pad 1: +BATT -> +3.3V
- R8 pad 2: Net-(U3-IO1) -> /wind_dir
- R9 pad 1: Net-(U3-IO1) -> +3.3V
- R9 pad 2: GND -> /rain_sensor
- U1 pad 1: Net-(U1-EN) -> unconnected-(U1-32KHZ-Pad1)
- U1 pad 2: GND -> I2C_PWR
- U1 pad 3: Net-(U1-FB) -> /IRQ_DS
- U1 pad 4: Net-(U1-FB) -> /RST_DS
- U1 pad 5: Net-(U1-FB) -> GND
- U1 pad 6: Net-(L1-Pad2) -> Net-(BT1-+)
- U1 pad 7: Net-(L1-Pad2) -> /SDA
- U1 pad 8: Net-(L1-Pad1) -> /SCL
- U2 pad 1: VS -> unconnected-(U2-ANT-Pad1)
- U2 pad 10: Net-(U2-VIN) -> unconnected-(U2-DIO4-Pad10)
- U2 pad 11: (no net) -> unconnected-(U2-DIO5-Pad11)
- U2 pad 2: +BATT -> GND
- U2 pad 3: Net-(U2-STAT2) -> Lora_PWR
- U2 pad 4: GND -> /RST_Lora
- U2 pad 5: GND -> /IRQ_Lora
- U2 pad 6: /THERM -> unconnected-(U2-DIO1-Pad6)
- U2 pad 7: /ILIM/VSET -> unconnected-(U2-DIO2-Pad7)
- U2 pad 8: /ISET -> unconnected-(U2-DIO3-Pad8)
- U2 pad 9: Net-(U2-STAT1) -> GND
- U3 pad 1: GND -> /D+
- U3 pad 2: +3.3V -> GND
- U3 pad 3: /Reset -> /D-
- U3 pad 4: unconnected-(U3-IO4-Pad4) -> /USB_D-
- U3 pad 5: unconnected-(U3-IO5-Pad5) -> VBUS
- U3 pad 6: unconnected-(U3-IO6-Pad6) -> /USB_D+
- U4 pad 1: unconnected-(U4-ANT-Pad1) -> GND
- U4 pad 10: unconnected-(U4-DIO4-Pad10) -> /Btn_User
- U4 pad 11: unconnected-(U4-DIO5-Pad11) -> /RST_Lora
- U4 pad 12: unconnected-(U4-SCK-Pad12) -> /SDA
- U4 pad 13: unconnected-(U4-MISO-Pad13) -> /USB_D-
- U4 pad 14: unconnected-(U4-MOSI-Pad14) -> /USB_D+
- U4 pad 16: GND -> unconnected-(U4-IO46-Pad16)
- U4 pad 2: GND -> +3.3V
- U4 pad 3: +3.3V -> /Reset
- U4 pad 5: unconnected-(U4-DIO0-Pad5) -> /cmd_Lora_PWR
- U4 pad 6: unconnected-(U4-DIO1-Pad6) -> LED_PWR
- U4 pad 7: unconnected-(U4-DIO2-Pad7) -> /cmd_I2C_PWR
- U4 pad 8: unconnected-(U4-DIO3-Pad8) -> /rain_sensor
- U4 pad 9: GND -> /wind_speed
- U5 pad 1: unconnected-(U5-32KHZ-Pad1) -> Net-(U5-EN)
- U5 pad 2: +3.3V -> GND
- U5 pad 3: unconnected-(U5-~{INT}/SQW-Pad3) -> Net-(U5-FB)
- U5 pad 4: unconnected-(U5-~{RST}-Pad4) -> Net-(U5-FB)
- U5 pad 5: GND -> Net-(U5-FB)
- U5 pad 6: Net-(BT1-+) -> Net-(L1-Pad2)
- U5 pad 7: /SDA -> Net-(L1-Pad2)
- U5 pad 8: /SCL -> Net-(L1-Pad1)
Other:
- board outline added: 88.5 x 71.5 mm
