File: power.kicad_sch (KiCad schematic)
At the start: 43 parts, among them J1 Solar connector, J2 JST2PH Batt LiFePo4 3.2v, Q1 IRLML6401, Q2 IRLML6401, Q3 IRLML6401, U1 TPS63021, U2 BQ25185

Commit message: update footprints
Parts:
- C10: renamed from C3; footprint (none) -> Capacitor_SMD:C_1206_3216Metric_Pad1.33x1.80mm_HandSolder
- C11: renamed from C1; footprint (none) -> Capacitor_SMD:C_1206_3216Metric_Pad1.33x1.80mm_HandSolder
- C12: renamed from C2; footprint (none) -> Capacitor_SMD:C_1206_3216Metric_Pad1.33x1.80mm_HandSolder
- C14: renamed from C7; footprint (none) -> Capacitor_SMD:C_1210_3225Metric_Pad1.33x2.70mm_HandSolder
- C15: renamed from C8; footprint (none) -> Capacitor_SMD:C_1210_3225Metric_Pad1.33x2.70mm_HandSolder
- C16: renamed from C9; footprint (none) -> Capacitor_SMD:C_1210_3225Metric_Pad1.33x2.70mm_HandSolder
- C17: renamed from C5; footprint (none) -> Capacitor_SMD:C_1210_3225Metric_Pad1.33x2.70mm_HandSolder
- C18: renamed from C6; footprint (none) -> Capacitor_SMD:C_1210_3225Metric_Pad1.33x2.70mm_HandSolder
- C19: renamed from C18; footprint (none) -> Capacitor_SMD:C_1210_3225Metric_Pad1.33x2.70mm_HandSolder
- F1, F2, F3, F4: footprint (none) -> Fuse:Fuse_1206_3216Metric
- renumbered C4 to C13, D9 to D10, D6 to D11, D7 to D12, D10 to D13, D1 to D6, D2 to D7, D4 to D8, D5 to D9, J2 to J8, J1 to J9, R6 to R12, R7 to R13, R13 to R14, R14 to R15, R12 to R16, R15 to R17, R2 to R18, R3 to R19, R22 to R20, R8 to R21, R9 to R22, U1 to U5, U2 to U6
Other:
- note added: "High Efficiency Single Inductor Buck-Boost Converter with 4A Switch"

Commit message: update schema
set the correct ESP32 pins
Parts:
- added TP10: I2C_PWR, TestPoint:TestPoint_Pad_D2.0mm, symbol Connector:TestPoint
- added TP11: Lora_PWR, TestPoint:TestPoint_Pad_D2.0mm, symbol Connector:TestPoint
- added TP6: Solar, TestPoint:TestPoint_Pad_D2.0mm, symbol Connector:TestPoint
- added TP7: VBatt, TestPoint:TestPoint_Pad_D2.0mm, symbol Connector:TestPoint
- added TP8: 3.3V, TestPoint:TestPoint_Pad_D2.0mm, symbol Connector:TestPoint
- added TP9: SD_PWR, TestPoint:TestPoint_Pad_D2.0mm, symbol Connector:TestPoint
Connections:
- net +BATT: now also TP7.1
- net I2C_PWR: now also TP10.1
- net Lora_PWR: now also TP11.1
- net SD_PWR: now also TP9.1
- net at C10.1, D6.A, J9.2 (Pin_2): now also TP6.1
- net at C14.1, C15.1, C16.1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: now also TP8.1

Commit message: update schematic
finalize
Parts:
- removed C14: 22uF, Capacitor_SMD:C_1210_3225Metric_Pad1.33x2.70mm_HandSolder, symbol Device:C
- removed TP6: Solar, TestPoint:TestPoint_Pad_D2.0mm, symbol Connector:TestPoint
- added C16: 22uF, Capacitor_SMD:C_1210_3225Metric_Pad1.33x2.70mm_HandSolder, symbol Device:C
- added C18: 22uF, Capacitor_SMD:C_Elec_5x5.4, symbol Device:C_Polarized_US
- renumbered C10 to C11, C11 to C12, C12 to C13, C13 to C14, C16 to C17, C17 to C19, C18 to C20, C19 to C21, R17 to R16, R16 to R17, TP11 to TP10, TP7 to TP6, TP8 to TP7, TP9 to TP8, TP10 to TP9
Connections:
- net +3.3V: now also C18.1
- net GND: now also C16.2, C18.2
- net at C15.1, C17.1, FB1.1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: now also C16.1
Other:
- moved on the sheet: D10, R17

Commit message: clean schematic
Check ERC error ok
Parts:
- removed D6, D7: NSR0320, Diode_SMD:D_SOD-323_HandSoldering, symbol lifepo4_solar_charger-eagle-import:DIODE_SOD323MINI
- removed U6: BQ25185, Package_SON:WSON-10-1EP_2.5x2.5mm_P0.5mm_EP1.2x2mm_ThermalVias, symbol lifepo4_solar_charger-eagle-import:BQ25185
- added D6, D7: NSR0320, Diode_SMD:D_SOD-323_HandSoldering, symbol Device:D
- added U6: BQ25185, Package_SON:WSON-10-1EP_2.5x2.5mm_P0.5mm_EP1.2x2mm_ThermalVias, symbol mSolarLib:BQ25185
- FB1: footprint Inductor_SMD:L_0805_2012Metric_Pad1.15x1.40mm_HandSolder -> Inductor_SMD:L_0805_2012Metric_Pad1.05x1.20mm_HandSolder; Fournisseur RS: 724-1542 -> (none); ref (none) -> RS: 724-1542
- renumbered J8 to J10, J9 to J11, TP6 to TP1, TP7 to TP2, TP8 to TP3, TP9 to TP4, TP10 to TP5
Connections:
- net +BATT: now also U6.2 (VBAT)
- net GND: now also U6.4 (/CE), U6.5 (GND), U6.PAD (GND)
- net ILIM/VSET: now also U6.7 (VSET)
- net ISET: now also U6.8 (ISET)
- net THERM: now also U6.6 (TS/MR)
- net VBUS: now also D7.2 (A)
- net VS: now also U6.1 (VSYS)
- net at C11.1, J11.2 (Pin_2): now also D6.2 (A)
- net at R12.2: now also U6.9 (STAT1)
- net at R13.2: now also U6.3 (STAT2)
- new net: D6.1 (K), D7.1 (K), U6.10 (VIN)

Commit message: update and starting PCB
Parts:
- D10: Fournisseur RS: 914-8619 -> (none); ref (none) -> VLMC3100-GS08
- D8: Fournisseur RS: 914-8619 -> (none); ref (none) -> VLMS30K1L2-GS08
- F1: ref (none) -> 1206L260SLTHYR
- F2, F3, F4: ref (none) -> 1206L150/12SLYR
- L1: footprint Inductor_SMD_Wurth:L_Wurth_WE-LQSH-2010 -> Inductor_SMD_Wurth:L_Wurth_WE-LQSH-4020; Mouser (none) -> VLS3015CX-1R5M-H
Connections:
- net GND: now also U6.11 (Thermal)
- net I2C_PWR: now also C20.1
- net Lora_PWR: now also C21.1
- net SD_PWR: now also C19.1
- net at F4.1, Q3.3 (D): no longer C21.1
- net at F2.1, Q1.3 (D): no longer C19.1
- net at F3.1, Q2.3 (D): no longer C20.1
Other:
- moved on the sheet: C19, D11, F2, R21, TP3, TP4, TP5
